Commit message: [update]

File: vicpinky_description/urdf/camera.xacro (robot description, xacro)
@@ -1,25 +1,56 @@
 <?xml version="1.0"?>
 <robot xmlns:xacro="http://www.ros.org/wiki/xacro" >
-    <gazebo reference="camera_link">
-        <sensor name="camera" type="camera">
+    <xacro:arg name="namespace" default=""/>
+    <xacro:property name="prefix" value="$(arg namespace)"/>
+    <!-- Orbbec Astra RGB Camera -->
+    <gazebo reference="${prefix}camera_link">
+        <sensor name="astra_rgb_camera" type="camera">
             <always_on>true</always_on>
             <visualize>true</visualize>
             <update_rate>30</update_rate>
-            <topic>camera/image_raw</topic>
-            <gz_frame_id>camera_rgb_frame</gz_frame_id>
-            <camera name="intel_realsense_r200">
-                <camera_info_topic>camera/camera_info</camera_info_topic>
-                <horizontal_fov>1.08</horizontal_fov>
+            <topic>${prefix}camera/color/image_raw</topic>
+            <gz_frame_id>${prefix}camera_color_frame</gz_frame_id>
+            <camera name="orbbec_astra">
+                <camera_info_topic>${prefix}camera/color/camera_info</camera_info_topic>
+                <horizontal_fov>1.02</horizontal_fov>
                 <image>
-                    <width>1280</width>
-                    <height>720</height>
+                    <width>640</width>
+                    <height>480</height>
                     <format>R8G8B8</format>
                 </image>
                 <clip>
                     <near>0.02</near>
-                    <far>300</far>
+                    <far>10.0</far>
                 </clip>
                 <noise>
-                <type>gaussian</type>
+                    <type>gaussian</type>
+                    <mean>0.0</mean>
+                    <stddev>0.007</stddev>
+                </noise>
+            </camera>
+        </sensor>
+    </gazebo>
+    <!-- Orbbec Astra Depth Camera -->
+    <gazebo reference="${prefix}camera_link">
+        <sensor name="astra_depth_camera" type="depth_camera">
+            <always_on>true</always_on>
+            <visualize>true</visualize>
+            <update_rate>30</update_rate>
+            <topic>${prefix}camera/depth/image_raw</topic>
+            <gz_frame_id>${prefix}camera_depth_frame</gz_frame_id>
+            <camera name="orbbec_astra_depth">
+                <camera_info_topic>${prefix}camera/depth/camera_info</camera_info_topic>
+                <horizontal_fov>1.02</horizontal_fov>
+                <image>
+                    <width>640</width>
+                    <height>480</height>
+                    <format>R_FLOAT32</format>
+                </image>
+                <clip>
+                    <near>0.1</near>
+                    <far>10.0</far>
+                </clip>
+                <noise>
+                    <type>gaussian</type>
                     <mean>0.0</mean>
                     <stddev>0.01</stddev>

File: vicpinky_description/urdf/robot_core.xacro (robot description, xacro)
@@ -235,3 +235,55 @@
         <origin xyz="0.0 0 0.03" rpy="0 0 ${pi}"/>
     </joint>
+    <!-- Orbbec Astra Camera Mount -->
+    <link name="${prefix}camera_mount">
+        <visual>
+            <origin xyz="0 0 0" rpy="0 0 0"/>
+            <geometry>
+                <box size="0.06 0.08 0.04"/>
+            </geometry>
+            <material name="gray"/>
+        </visual>
+        <collision>
+            <origin xyz="0 0 0" rpy="0 0 0"/>
+            <geometry>
+                <box size="0.06 0.08 0.04"/>
+            </geometry>
+        </collision>
+        <xacro:inertial_box mass="0.05" x="0.06" y="0.08" z="0.04">
+            <origin xyz="0 0 0" rpy="0 0 0"/>
+        </xacro:inertial_box>
+    </link>
+    <joint name="${prefix}camera_mount_fixed_joint" type="fixed">
+        <parent link="${prefix}base_link"/>
+        <child link="${prefix}camera_mount"/>
+        <origin xyz="-0.29 0 1.27" rpy="0 0 0"/>
+    </joint>
+    <!-- Orbbec Astra Camera Link -->
+    <link name="${prefix}camera_link"/>
+    <joint name="${prefix}camera_link_fixed_joint" type="fixed">
+        <parent link="${prefix}camera_mount"/>
+        <child link="${prefix}camera_link"/>
+        <origin xyz="0.03 0 0" rpy="0 0 0"/>
+    </joint>
+    <!-- Camera RGB Frame -->
+    <link name="${prefix}camera_rgb_frame"/>
+    <joint name="${prefix}camera_rgb_joint" type="fixed">
+        <parent link="${prefix}camera_link"/>
+        <child link="${prefix}camera_rgb_frame"/>
+        <origin xyz="0 0 0" rpy="0 0 0"/>
+    </joint>
+    <!-- Camera Depth Frame -->
+    <link name="${prefix}camera_depth_frame"/>
+    <joint name="${prefix}camera_depth_joint" type="fixed">
+        <parent link="${prefix}camera_link"/>
+        <child link="${prefix}camera_depth_frame"/>
+        <origin xyz="0 0 0" rpy="0 0 0"/>
+    </joint>
+    <!-- Camera Color Frame (for compatibility) -->
+    <link name="${prefix}camera_color_frame"/>
+    <joint name="${prefix}camera_color_joint" type="fixed">
+        <parent link="${prefix}camera_link"/>
+        <child link="${prefix}camera_color_frame"/>
+        <origin xyz="0 0 0" rpy="0 0 0"/>
+    </joint>
 </robot>
